File: hw/haier-controller.kicad_pcb (KiCad board)
At the start: 2 copper layers, 95 parts, among them J1 USB4105-GF-A, J10 DG240W, J11 DG240W, J12 DG240W, J2 10118194-0001LF, J3 TC2050-IDC-NL, J4 Goldpin, J5 BM04B, J6 S3B-XH-A-1, J7 S3B-XH-A-1, J8 S4B-XH-A-1, J9 S4B-XH-A-1, K1 HFD27-005-S, K2 HFD23/005-1ZS, K3 HFD23/005-1ZS, K4 HFD23/005-1ZS, Q1 MMBT3904, Q2 MMBT3904, Q3 MMBT3904, Q4 MMBT3904, Q5 MMBT3904, SW1 PTS526SM15SMTR2_LFS, U1 ESP32-C6, U2 LM66200DRLR, U3 LD1117S33CTR, U4 USBLC6-4SC6, U5 DS2401+, U6 MAX3485EESA+T

Commit message: Finish PCB
Parts:
- added H1: M3, mechanical:M3-Hole, F.Cu at (92.5, 126.0)
- added H2: M3, mechanical:M3-Hole, F.Cu at (62.5, 85.0)
- added H3: M3, mechanical:M3-Hole, F.Cu at (133.5, 85.0)
- added H4: M3, mechanical:M3-Hole, F.Cu at (133.5, 131.0)
- J3: value TC2050-IDC-NL -> FTSH-105-01-L-DV-K; footprint connectors:TC2050-IDC-NL -> connectors:FTSH-105-01-L-DV-K
- R1, R3: footprint SMD:C_0603 -> SMD:R_0603
- moved R3 97.7 mm to (68.1, 142.4), turned to 180 degrees
- moved C2 96.5 mm to (67.3, 147.0), turned to 90 degrees
- moved C1 92.3 mm to (67.3, 140.0), turned to -90 degrees
- moved J8 87.3 mm to (123.0, 140.6)
- moved R1 86.0 mm to (68.1, 144.6), turned to 180 degrees
- moved C10 86.0 mm to (79.5, 137.0), turned to 180 degrees
- moved C3 83.6 mm to (64.7, 133.0), turned to 90 degrees
- moved C5 81.5 mm to (70.8, 138.7)
- moved R2 80.4 mm to (73.4, 143.4), turned to -90 degrees
- moved C4 79.7 mm to (70.8, 134.4)
- moved R4 79.3 mm to (68.3, 122.5)
- moved R5 76.6 mm to (70.7, 123.3), turned to -90 degrees
- moved C14 76.0 mm to (67.2, 125.0), turned to 90 degrees
- moved R7 75.4 mm to (88.5, 136.7), turned to 180 degrees
- moved C6 75.3 mm to (74.2, 135.7), turned to -90 degrees
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Connections:
- C1 pad 1: Net-(C1-Pad1) -> GND
- C1 pad 2: VBUS -> VBUS_A
- C10 pad 1: Net-(C10-Pad1) -> GND
- C10 pad 2: Net-(U3-VOUT) -> +3.3V
- C11 pad 1: Net-(C11-Pad1) -> GND
- C11 pad 2: Net-(U1-3V3) -> +3.3V
- C12 pad 1: Net-(C12-Pad1) -> GND
- C12 pad 2: Net-(U1-3V3) -> +3.3V
- C13 pad 1: Net-(C13-Pad1) -> GND
- C14 pad 1: Net-(C14-Pad1) -> GND
- C15 pad 1: Net-(U4-GND) -> GND
- C15 pad 2: Net-(U4-VBUS) -> +3.3V
- C16 pad 1: Net-(U6-VCC) -> +3.3V
- C16 pad 2: Net-(C16-Pad2) -> GND
- C2 pad 1: Net-(C1-Pad1) -> GND
- C2 pad 2: VBUS -> VBUS_A
- C3 pad 1: Net-(C3-Pad1) -> GND
- C3 pad 2: Net-(J2-VCC) -> VBUS_B
- C4 pad 1: Net-(C4-Pad1) -> GND
- C4 pad 2: Net-(U2-VIN1) -> VBUS_B
- C5 pad 1: Net-(C5-Pad1) -> GND
- C5 pad 2: Net-(U2-VIN2) -> VBUS_A
- C6 pad 1: Net-(C6-Pad1) -> GND
- C6 pad 2: Net-(U3-VIN) -> VBUS
- C7 pad 1: Net-(C6-Pad1) -> GND
- C7 pad 2: Net-(U3-VIN) -> VBUS
- C8 pad 1: Net-(C8-Pad1) -> GND
- C8 pad 2: Net-(U3-VIN) -> VBUS
- C9 pad 1: Net-(C9-Pad1) -> GND
- C9 pad 2: Net-(U3-VOUT) -> +3.3V
- D1 pad 1: Net-(D1-Pad1) -> GND
- D10 pad 1: Net-(K2-GND) -> VBUS
- D11 pad 1: Net-(K3-GND) -> VBUS
- D12 pad 1: Net-(K4-GND) -> VBUS
- D2 pad 1: Net-(D2-Pad1) -> GND
- D3 pad 1: Net-(D3-Pad1) -> GND
- D4 pad 1: Net-(D4-Pad1) -> GND
- D5 pad 1: Net-(D5-Pad1) -> GND
- D6 pad 2: Net-(D6-Pad2) -> GND
- D8 pad 1: Net-(D8-Pad1) -> GND
- D9 pad 1: Net-(K1-GND) -> VBUS
- J1 pad A1: Net-(J1-Shield) -> GND
- J1 pad A12: Net-(J1-Shield) -> GND
- J1 pad A4: VBUS -> VBUS_A
- J1 pad A9: VBUS -> VBUS_A
- J1 pad SH: Net-(J1-Shield) -> GND
- J10 pad 1: Net-(J10-Pad1) -> Net-(K2-NO1)
- J10 pad 2: Net-(K2-NO1) -> Net-(J10-Pad2)
- J11 pad 1: Net-(J11-Pad1) -> Net-(K3-NO1)
- J11 pad 2: Net-(K3-NO1) -> Net-(J11-Pad2)
- J12 pad 1: Net-(J12-Pad1) -> Net-(K4-NO1)
- J12 pad 2: Net-(K4-NO1) -> Net-(J12-Pad2)
- J2 pad 1: Net-(J2-VCC) -> VBUS_B
- J2 pad 5: Net-(J2-GND) -> GND
- J2 pad SH: Net-(J2-GND) -> GND
- J3 pad 1: Net-(J3-VTRef) -> +3.3V
- J3 pad 3: Net-(J3-GND-Pad3) -> GND
- J3 pad 5: Net-(J3-GND-Pad3) -> GND
- J3 pad 7: unconnected-(J3-RTCLK-Pad7) -> GND
- J3 pad 9: unconnected-(J3-NTRST-Pad9) -> GND
- J4 pad 2: Net-(J4-Pad2) -> GND
- J5 pad 1: Net-(J5-Pad1) -> +3.3V
- J5 pad 4: Net-(J5-Pad4) -> GND
- J5 pad SH: Net-(J5-Pad4) -> GND
- J6 pad 2: Net-(J6-Pad2) -> GND
- J6 pad 3: Net-(J6-Pad3) -> +3.3V
- J7 pad 2: Net-(J7-Pad2) -> GND
- J7 pad 3: Net-(J7-Pad3) -> +3.3V
- K1 pad 8: Net-(K1-GND) -> VBUS
- K2 pad 3: Net-(J10-Pad1) -> Net-(J10-Pad2)
- K2 pad 4: Net-(J10-Pad1) -> Net-(J10-Pad2)
- K2 pad 5: Net-(K2-GND) -> VBUS
- K3 pad 3: Net-(J11-Pad1) -> Net-(J11-Pad2)
- K3 pad 4: Net-(J11-Pad1) -> Net-(J11-Pad2)
- K3 pad 5: Net-(K3-GND) -> VBUS
- K4 pad 3: Net-(J12-Pad1) -> Net-(J12-Pad2)
- K4 pad 4: Net-(J12-Pad1) -> Net-(J12-Pad2)
- K4 pad 5: Net-(K4-GND) -> VBUS
- Q1 pad 3: Net-(Q1-E) -> GND
- Q2 pad 3: Net-(Q2-E) -> GND
- Q3 pad 3: Net-(Q3-E) -> GND
- Q4 pad 3: Net-(Q4-E) -> GND
- Q5 pad 3: Net-(Q5-E) -> GND
- R1 pad 1: Net-(C1-Pad1) -> GND
- R11 pad 1: Net-(R11-Pad1) -> +3.3V
- R12 pad 2: Net-(R12-Pad2) -> GND
- R13 pad 2: Net-(R13-Pad2) -> GND
- R14 pad 1: Net-(R14-Pad1) -> +3.3V
- R2 pad 1: Net-(U3-VIN) -> VBUS
- R20 pad 2: Net-(K4-GND) -> VBUS
- R21 pad 2: Net-(K3-GND) -> VBUS
- R22 pad 2: Net-(K2-GND) -> VBUS
- R23 pad 2: Net-(K1-GND) -> VBUS
- R3 pad 1: Net-(C1-Pad1) -> GND
- R4 pad 1: Net-(R4-Pad1) -> +3.3V
- R6 pad 2: Net-(R6-Pad2) -> +3.3V
- R7 pad 1: Net-(J6-Pad3) -> +3.3V
- R8 pad 1: Net-(J7-Pad3) -> +3.3V
- R9 pad 1: Net-(U1-IO18) -> Net-(U1-IO10)
- SW1 pad 2: Net-(C14-Pad1) -> GND
- TP1 pad 1: Net-(J2-VCC) -> VBUS_B
- TP2 pad 1: VBUS -> VBUS_A
- TP3 pad 1: Net-(U3-VIN) -> VBUS
- TP4 pad 1: Net-(U3-VOUT) -> +3.3V
- TP6 pad 1: Net-(J1-Shield) -> GND
- U1 pad 1: Net-(U1-EPAD) -> GND
- U1 pad 11: /COOL_SW -> Net-(U1-IO10)
- U1 pad 12: /LIM_SW -> /RS_SWITCH
- U1 pad 13: unconnected-(U1-IO12-Pad13) -> /DS18B20
- U1 pad 14: unconnected-(U1-IO13-Pad14) -> /1W_ID
- U1 pad 16: Net-(U1-IO18) -> /LIM_SW
- U1 pad 17: unconnected-(U1-IO19-Pad17) -> /COOL_SW
- U1 pad 18: unconnected-(U1-IO20-Pad18) -> /HEAT_SW
- U1 pad 2: Net-(U1-3V3) -> +3.3V
- U1 pad 26: /HEAT_SW -> unconnected-(U1-IO3-Pad26)
- U1 pad 27: /RS_SWITCH -> unconnected-(U1-IO2-Pad27)
- U1 pad 28: Net-(U1-EPAD) -> GND
- U1 pad 29: Net-(U1-EPAD) -> GND
- U1 pad 8: /DS18B20 -> unconnected-(U1-IO0-Pad8)
- U1 pad 9: /1W_ID -> unconnected-(U1-IO1-Pad9)
- U2 pad 1: Net-(U2-GND-Pad1) -> GND
- U2 pad 2: Net-(U3-VIN) -> VBUS
- U2 pad 3: Net-(U2-VIN1) -> VBUS_B
- U2 pad 4: Net-(U2-~{ON}) -> GND
- U2 pad 5: Net-(U2-GND-Pad1) -> GND
- U2 pad 6: Net-(U2-VIN2) -> VBUS_A
- U2 pad 7: Net-(U3-VIN) -> VBUS
- U3 pad 1: Net-(U3-GND) -> GND
- U3 pad 2: Net-(U3-VOUT) -> +3.3V
- U3 pad 3: Net-(U3-VIN) -> VBUS
- U4 pad 2: Net-(U4-GND) -> GND
- U4 pad 4: /ESP_TDO -> /ESP_TDI
- U4 pad 5: Net-(U4-VBUS) -> +3.3V
- U4 pad 6: /ESP_TDI -> /ESP_TDO
- U5 pad 1: Net-(U5-GND) -> GND
- U6 pad 5: Net-(U6-GND) -> GND
- U6 pad 8: Net-(U6-VCC) -> +3.3V
Routing:
- net +3.3V: track 0.00 -> 214.9 mm, vias 0 -> 2
- net VBUS: track 0.00 -> 211.2 mm, vias 0 -> 2
- net GND: track 0.00 -> 81.9 mm, vias 0 -> 56
- net Net-(K1-VCC): track 0.00 -> 69.4 mm, vias 0 -> 2
- net Net-(K2-VCC): track 0.00 -> 66.3 mm
- net /PUMP_RX: track 0.00 -> 65.3 mm
- net /PUMP_TX: track 0.00 -> 58.7 mm
- net /HEAT_SW: track 0.00 -> 56.0 mm
- net Net-(K3-VCC): track 0.00 -> 54.0 mm
- net Net-(K4-VCC): track 0.00 -> 44.8 mm
- net /1W_ID: track 0.00 -> 44.0 mm
- net /COOL_SW: track 0.00 -> 39.9 mm
- net /PUMP_A: track 0.00 -> 37.3 mm
- net /PUMP_B: track 0.00 -> 36.0 mm
- net /ESP_EN: track 0.00 -> 33.4 mm
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- added copper zone on B.Cu, net GND
Other:
- board outline added: 79 x 70 mm

Commit message: Update components, Add silkscreen descriptors
Parts:
- C12: value 22u -> 22uF
- turned R16 to -90 degrees
- turned R17 to 90 degrees
- turned R18 to 90 degrees
- turned R19 to 90 degrees
- turned R20 to 90 degrees
- turned R21 to 90 degrees
- turned R22 to 90 degrees
- turned R23 to 90 degrees
- turned R9 to 90 degrees
Connections:
- R16 pad 1: /RS_SWITCH -> Net-(Q2-B)
- R16 pad 2: Net-(Q2-B) -> /RS_SWITCH
- R17 pad 1: /HEAT_SW -> Net-(Q3-B)
- R17 pad 2: Net-(Q3-B) -> /HEAT_SW
- R18 pad 1: /COOL_SW -> Net-(Q4-B)
- R18 pad 2: Net-(Q4-B) -> /COOL_SW
- R19 pad 1: /LIM_SW -> Net-(Q5-B)
- R19 pad 2: Net-(Q5-B) -> /LIM_SW
- R20 pad 1: Net-(D13-Pad2) -> VBUS
- R20 pad 2: VBUS -> Net-(D13-Pad2)
- R21 pad 1: Net-(D14-Pad2) -> VBUS
- R21 pad 2: VBUS -> Net-(D14-Pad2)
- R22 pad 1: Net-(D15-Pad2) -> VBUS
- R22 pad 2: VBUS -> Net-(D15-Pad2)
- R23 pad 1: Net-(D16-Pad2) -> VBUS
- R23 pad 2: VBUS -> Net-(D16-Pad2)
- R9 pad 1: Net-(U1-IO10) -> Net-(D5-Pad2)
- R9 pad 2: Net-(D5-Pad2) -> Net-(U1-IO10)
Other:
- board text added: "3V3"
- board text added: "COOL"
- board text added: "DRIVER"
- board text added: "DRV"
- board text added: "DS18B20"
- board text added: "DS2401+"
- board text added: "EN"
- board text added: "GND"
- board text added: "HEAT"
- board text added: "ID"
- board text added: "LIM"
- board text added: "LIMIT"
- board text added: "MRWorkshop Haier-controller Rev. 1.0.0 07/26"
- board text added: "PUMP"
- board text added: "PUMP_A"
- board text added: "PUMP_B"
- board text added: "RST"
- board text added: "RX"
- board text added: "TEMP"
- board text added: "TX"
- board text added: "UART"
- board text added: "VA"
- board text added: "VB"
- board text added: "VBUS"
