File: hw/haier-controller.kicad_pcb (KiCad board)
At the start: 2 copper layers, 79 x 70 mm, 99 parts, among them J1 USB4105-GF-A, J10 DG240W, J11 DG240W, J12 DG240W, J2 10118194-0001LF, J3 FTSH-105-01-L-DV-K, J4 Goldpin, J5 BM04B, J6 S3B-XH-A-1, J7 S3B-XH-A-1, J8 S4B-XH-A-1, J9 S4B-XH-A-1, K1 HFD27-005-S, K2 HFD23/005-1ZS, K3 HFD23/005-1ZS, K4 HFD23/005-1ZS, Q1 MMBT3904, Q2 MMBT3904, Q3 MMBT3904, Q4 MMBT3904, Q5 MMBT3904, SW1 PTS526SM15SMTR2_LFS, U1 ESP32-C6, U2 LM66200DRLR, U3 LD1117S33CTR, U4 USBLC6-4SC6, U5 DS2401+, U6 MAX3485EESA+T

Commit message: Update PCB
Parts:
- added R24: 10k, SMD:R_0603, F.Cu at (97.5, 107.0)
- added R25: 10k, SMD:R_0603, F.Cu at (111.2, 107.0)
- added R26: 10k, SMD:R_0603, F.Cu at (125.2, 107.0)
- added R27: 10k, SMD:R_0603, F.Cu at (98.7, 128.7)
- added R28: 0R, SMD:R_0603, F.Cu at (72.4, 140.3)
- added R29: 0R, SMD:R_0603, F.Cu at (68.3, 136.5)
- moved TP1 7.06 mm to (72.8, 131.6)
Routing:
- net VBUS: track 211.2 -> 218.6 mm
- net GND: track 81.9 -> 87.1 mm, vias 56 -> 60
- net VBUS_B: track 15.8 -> 18.7 mm
- net /RS_SWITCH: track 29.1 -> 30.1 mm
